File: hardware/board/sniff_detector/harp_core_rp2040_w_isolated_usb.kicad_sch (KiCad schematic)
At the start: 49 parts, among them J2 Conn_01x03_Male, J4 AudioJack3, J5 USB_C_Receptacle_USB2.0, U2 TPD2EUSB30, U3 ADUM4160, U4 RP2040, U5 W25Q16JVUXIQ, X1 ECS-TXO-2016

Commit message: draft firmware
Parts:
- C10, C56, C8, C9: Tolerance (none) -> 10%; Voltage (none) -> 35V
- C11: footprint Capacitor_SMD:C_0805_2012Metric -> Capacitor_SMD:C_0603_1608Metric; Alternate CL21B106KOQNNNE -> (none); Link https://www.digikey.com/en/products/detail/murata-electronics/GRM21BZ71E106KE15L/13904911 -> https://www.digikey.com/en/products/detail/murata-electronics/GRM188R61E106KA73J/9887674; Manufacturer Number GRM21BZ71E106KE15L -> GRM188R61E106KA73J; Temperature Coefficient X7R -> X5R; Tolerance (none) -> 10%; Voltage (none) -> 25V
- C32: Voltage (none) -> 25V
- J4: Alternate SJ-3523-SMT-TR -> (none); Link https://www.digikey.com/en/products/detail/cui-devices/SJ-3524-SMT-TR-BE/2295987 -> https://www.digikey.com/en/products/detail/cui-devices/SJ-3523-SMT-TR/281297; Manufacturer Number SJ-3524-SMT-TR-BE -> SJ-3523-SMT-TR
Changed lines of the file:
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@@
       (effects (font (size 1.27 1.27)) hide)
     )
+    (property "Voltage" "25V" (at 31.75 184.785 0)
+      (effects (font (size 1.27 1.27)) hide)
+    )
     (pin "1")
     (pin "2")
@@
       (effects (font (size 1.27 1.27)) hide)
     )
+    (property "Voltage" "35V" (at 59.69 184.785 0)
+      (effects (font (size 1.27 1.27)) hide)
+    )
+    (property "Tolerance" "10%" (at 59.69 184.785 0)
+      (effects (font (size 1.27 1.27)) hide)
+    )
     (pin "1")
     (pin "2")
@@
       (effects (font (size 1.27 1.27)) hide)
     )
+    (property "Voltage" "35V" (at 74.295 149.225 0)
+      (effects (font (size 1.27 1.27)) hide)
+    )
+    (property "Tolerance" "10%" (at 74.295 149.225 0)
+      (effects (font (size 1.27 1.27)) hide)
+    )
     (pin "1")
     (pin "2")
@@
       (effects (font (size 1.27 1.27)) hide)
     )
-    (property "Link" "https://www.digikey.com/en/products/detail/cui-devices/SJ-3524-SMT-TR-BE/2295987" (at 24.13 121.285 0)
+    (property "Link" "https://www.digikey.com/en/products/detail/cui-devices/SJ-3523-SMT-TR/281297" (at 24.13 121.285 0)
       (effects (font (size 1.27 1.27)) hide)
     )
@@
       (effects (font (size 1.27 1.27)) hide)
     )
-    (property "Manufacturer Number" "SJ-3524-SMT-TR-BE" (at 24.13 121.285 0)
-      (effects (font (size 1.27 1.27)) hide)
-    )
-    (property "Alternate" "SJ-3523-SMT-TR" (at 24.13 121.285 0)
+    (property "Manufacturer Number" "SJ-3523-SMT-TR" (at 24.13 121.285 0)
       (effects (font (size 1.27 1.27)) hide)
     )
@@
       (effects (font (size 1.27 1.27)) hide)
     )
+    (property "Voltage" "35V" (at 78.74 184.785 0)
+      (effects (font (size 1.27 1.27)) hide)
+    )
+    (property "Tolerance" "10%" (at 78.74 184.785 0)
+      (effects (font (size 1.27 1.27)) hide)
+    )
     (pin "1")
     (pin "2")
@@
       (effects (font (size 1.27 1.27)) (justify left))
     )
-    (property "Footprint" "Capacitor_SMD:C_0805_2012Metric" (at 100.0252 188.595 0)
+    (property "Footprint" "Capacitor_SMD:C_0603_1608Metric" (at 100.0252 188.595 0)
       (effects (font (size 1.27 1.27)) hide)
     )
-    (property "Datasheet" "https://search.murata.co.jp/Ceramy/image/img/A01X/G101/ENG/GRM21BZ71E106KE15-01.pdf" (at 99.06 184.785 0)
+    (property "Datasheet" "https://search.murata.co.jp/Ceramy/image/img/A01X/G101/ENG/GRM188R61E106KA73-01A.pdf" (at 99.06 184.785 0)
       (effects (font (size 1.27 1.27)) hide)
     )
-    (property "Link" "https://www.digikey.com/en/products/detail/murata-electronics/GRM21BZ71E106KE15L/13904911" (at 99.06 184.785 0)
+    (property "Link" "https://www.digikey.com/en/products/detail/murata-electronics/GRM188R61E106KA73J/9887674" (at 99.06 184.785 0)
       (effects (font (size 1.27 1.27)) hide)
     )
-    (property "Manufacturer Number" "GRM21BZ71E106KE15L" (at 99.06 184.785 0)
+    (property "Manufacturer Number" "GRM188R61E106KA73J" (at 99.06 184.785 0)
       (effects (font (size 1.27 1.27)) hide)
     )
@@
       (effects (font (size 1.27 1.27)) hide)
     )
-    (property "Temperature Coefficient" "X7R" (at 99.06 184.785 0)
+    (property "Temperature Coefficient" "X5R" (at 99.06 184.785 0)
       (effects (font (size 1.27 1.27)) hide)
     )
@@
       (effects (font (size 1.27 1.27)) hide)
     )
-    (property "Alternate" "CL21B106KOQNNNE" (at 99.06 184.785 0)
+    (property "Alternate" "" (at 99.06 184.785 0)
+      (effects (font (size 1.27 1.27)) hide)
+    )
+    (property "Tolerance" "10%" (at 99.06 184.785 0)
+      (effects (font (size 1.27 1.27)) hide)
+    )
+    (property "Voltage" "25V" (at 99.06 184.785 0)
       (effects (font (size 1.27 1.27)) hide)
     )
@@
       (effects (font (size 1.27 1.27)) hide)
     )
+    (property "Voltage" "35V" (at 18.415 149.225 0)
+      (effects (font (size 1.27 1.27)) hide)
+    )
+    (property "Tolerance" "10%" (at 18.415 149.225 0)
+      (effects (font (size 1.27 1.27)) hide)
+    )
