File: hardware/board/sniff_detector/power_supplies.kicad_sch (KiCad schematic)
At the start: 21 parts, among them J6 Barrel_Jack_Switch, U9 LT3030

Commit message: draft firmware
Parts:
- C22, C23, C24: Voltage (none) -> 25V
- C25: footprint Capacitor_SMD:C_0805_2012Metric -> Capacitor_SMD:C_0603_1608Metric; Alternate CL21B106KOQNNNE -> (none); Link https://www.digikey.com/en/products/detail/murata-electronics/GRM21BZ71E106KE15L/13904911 -> https://www.digikey.com/en/products/detail/murata-electronics/GRM188R61E106KA73J/9887674; Manufacturer Number GRM21BZ71E106KE15L -> GRM188R61E106KA73J; Temperature Coefficient X7R -> X5R; Tolerance (none) -> 10%; Voltage (none) -> 25V
- C26: Manufacturer (none) -> Samsung Electro-Mechanics; Voltage (none) -> 25V
- C? (x3): footprint Resistor_SMD:R_0603_1608Metric -> Capacitor_SMD:C_0603_1608Metric; Rated Voltage (none) -> 25V; Temperature Coefficient (none) -> X5R; Vendor Number 490-GRM188R61E106KA73JDKR-ND -> (none)
Changed lines of the file:
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@@
+      (effects (font (size 1.27 1.27)) hide)
+    )
+    (property "Voltage" "25V" (at 105.41 53.34 0)
       (effects (font (size 1.27 1.27)) hide)
     )
@@
       (effects (font (size 1.27 1.27)) hide)
     )
+    (property "Voltage" "25V" (at 227.33 49.53 0)
+      (effects (font (size 1.27 1.27)) hide)
+    )
+    (property "Manufacturer" "Samsung Electro-Mechanics" (at 227.33 49.53 0)
+      (effects (font (size 1.27 1.27)) hide)
+    )
     (pin "1")
     (pin "2")
@@
       (effects (font (size 1.27 1.27)) (justify left))
     )
-    (property "Footprint" "Resistor_SMD:R_0603_1608Metric" (at 63.8302 188.595 0)
+    (property "Footprint" "Capacitor_SMD:C_0603_1608Metric" (at 63.8302 188.595 0)
       (effects (font (size 1.27 1.27)) hide)
     )
@@
       (effects (font (size 1.27 1.27)) hide)
     )
-    (property "Vendor Number" "490-GRM188R61E106KA73JDKR-ND" (at 62.865 184.785 0)
+    (property "Vendor Number" "" (at 62.865 184.785 0)
+      (effects (font (size 1.27 1.27)) hide)
+    )
+    (property "Rated Voltage" "25V" (at 62.865 184.785 0)
+      (effects (font (size 1.27 1.27)) hide)
+    )
+    (property "Temperature Coefficient" "X5R" (at 62.865 184.785 0)
       (effects (font (size 1.27 1.27)) hide)
     )
@@
     )
     (property "Tolerance" "10%" (at 156.21 45.72 0)
+      (effects (font (size 1.27 1.27)) hide)
+    )
+    (property "Voltage" "25V" (at 156.21 45.72 0)
       (effects (font (size 1.27 1.27)) hide)
     )
@@
       (effects (font (size 1.27 1.27)) (justify left))
     )
-    (property "Footprint" "Resistor_SMD:R_0603_1608Metric" (at 40.3352 188.595 0)
+    (property "Footprint" "Capacitor_SMD:C_0603_1608Metric" (at 40.3352 188.595 0)
       (effects (font (size 1.27 1.27)) hide)
     )
@@
       (effects (font (size 1.27 1.27)) hide)
     )
-    (property "Vendor Number" "490-GRM188R61E106KA73JDKR-ND" (at 39.37 184.785 0)
+    (property "Vendor Number" "" (at 39.37 184.785 0)
+      (effects (font (size 1.27 1.27)) hide)
+    )
+    (property "Rated Voltage" "25V" (at 39.37 184.785 0)
+      (effects (font (size 1.27 1.27)) hide)
+    )
+    (property "Temperature Coefficient" "X5R" (at 39.37 184.785 0)
       (effects (font (size 1.27 1.27)) hide)
     )
@@
       (effects (font (size 1.27 1.27)) (justify left))
     )
-    (property "Footprint" "Resistor_SMD:R_0603_1608Metric" (at 18.1102 188.595 0)
+    (property "Footprint" "Capacitor_SMD:C_0603_1608Metric" (at 18.1102 188.595 0)
       (effects (font (size 1.27 1.27)) hide)
     )
@@
       (effects (font (size 1.27 1.27)) hide)
     )
-    (property "Vendor Number" "490-GRM188R61E106KA73JDKR-ND" (at 17.145 184.785 0)
+    (property "Vendor Number" "" (at 17.145 184.785 0)
+      (effects (font (size 1.27 1.27)) hide)
+    )
+    (property "Rated Voltage" "25V" (at 17.145 184.785 0)
+      (effects (font (size 1.27 1.27)) hide)
+    )
+    (property "Temperature Coefficient" "X5R" (at 17.145 184.785 0)
       (effects (font (size 1.27 1.27)) hide)
     )
@@
       (effects (font (size 1.27 1.27)) hide)
     )
+    (property "Voltage" "25V" (at 156.21 60.96 0)
+      (effects (font (size 1.27 1.27)) hide)
+    )
     (pin "1")
     (pin "2")
@@
       (effects (font (size 1.27 1.27)) (justify left))
     )
-    (property "Footprint" "Capacitor_SMD:C_0805_2012Metric" (at 190.8302 68.58 0)
-      (effects (font (size 1.27 1.27)) hide)
-    )
-    (property "Datasheet" "https://search.murata.co.jp/Ceramy/image/img/A01X/G101/ENG/GRM21BZ71E106KE15-01.pdf" (at 189.865 64.77 0)
-      (effects (font (size 1.27 1.27)) hide)
-    )
-    (property "Link" "https://www.digikey.com/en/products/detail/murata-electronics/GRM21BZ71E106KE15L/13904911" (at 189.865 64.77 0)
-      (effects (font (size 1.27 1.27)) hide)
-    )
-    (property "Manufacturer Number" "GRM21BZ71E106KE15L" (at 189.865 64.77 0)
+    (property "Footprint" "Capacitor_SMD:C_0603_1608Metric" (at 190.8302 68.58 0)
+      (effects (font (size 1.27 1.27)) hide)
+    )
+    (property "Datasheet" "https://search.murata.co.jp/Ceramy/image/img/A01X/G101/ENG/GRM188R61E106KA73-01A.pdf" (at 189.865 64.77 0)
+      (effects (font (size 1.27 1.27)) hide)
+    )
+    (property "Link" "https://www.digikey.com/en/products/detail/murata-electronics/GRM188R61E106KA73J/9887674" (at 189.865 64.77 0)
+      (effects (font (size 1.27 1.27)) hide)
+    )
+    (property "Manufacturer Number" "GRM188R61E106KA73J" (at 189.865 64.77 0)
       (effects (font (size 1.27 1.27)) hide)
     )
@@
       (effects (font (size 1.27 1.27)) hide)
     )
-    (property "Temperature Coefficient" "X7R" (at 189.865 64.77 0)
+    (property "Temperature Coefficient" "X5R" (at 189.865 64.77 0)
       (effects (font (size 1.27 1.27)) hide)
     )
@@
       (effects (font (size 1.27 1.27)) hide)
     )
-    (property "Alternate" "CL21B106KOQNNNE" (at 189.865 64.77 0)
-      (effects (font (size 1.27 1.27)) hide)
-    )
+    (property "Alternate" "" (at 189.865 64.77 0)
+      (effects (font (size 1.27 1.27)) hide)
+    )
+    (property "Tolerance" "10%" (at 189.865 64.77 0)
+      (effects (font (size 1.27 1.27)) hide)
+    )
+    (property "Voltage" "25V" (at 189.865 64.77 0)
+      (effects (font (size 1.27 1.27)) hide)
+    )
