File: hardware/board/sniff_detector/sensing_front_end.kicad_sch (KiCad schematic)
At the start: 28 parts

Commit message: draft firmware
Parts:
- C?: Tolerance (none) -> 1%; Tolerlance 1% -> (none)
- C?: Voltage (none) -> 10V
- C?: footprint Capacitor_SMD:C_0402_1005Metric_Pad0.74x0.62mm_HandSolder -> Capacitor_SMD:C_0402_1005Metric; Link https://www.digikey.com/en/products/detail/samsung-electro-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 -> https://www.digikey.com/en/products/detail/murata-electroni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; Manufacturer Samsung Electro-Mechanics -> Murata Electronics; Manufacturer Number CL05A105KO5NNNC -> GRM155R6YA105KE11J; PCBWay Link https://www.pcbway.com/components/detail/CL05A105KO5NNNC/17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 -> (none); Rated Voltage (none) -> 35V; Temperature Coefficient (none) -> X5R; Tolerance 10% -> (none); Voltage 16V -> 35V
Other:
- note removed: "TODO: change out C34 to NP0? or change to 100nF if tolerance doesn't matter"
Changed lines of the file:
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@@
     (stroke (width 0) (type default))
   )
-  (wire (pts (xy 142.24 177.165) (xy 142.24 178.435))
+  (wire (pts (xy 142.24 175.895) (xy 142.24 178.435))
     (stroke (width 0) (type default))
   )
@@
     (stroke (width 0) (type default))
   )
-  (wire (pts (xy 88.9 177.165) (xy 88.9 178.435))
+  (wire (pts (xy 88.9 175.895) (xy 88.9 178.435))
     (stroke (width 0) (type default))
   )
@@
     (at 185.42 66.675 0)
     (effects (font (size 1.27 1.27)) (justify left bottom))
-  )
-  (text "TODO: change out C34 to NP0? or change to 100nF if tolerance doesn't matter"
-    (at 128.27 122.555 0)
-    (effects (font (size 2 2) (thickness 0.254) bold) (justify left bottom))
   )
   (text "i_{out,max} = 150[mA]" (at 175.26 71.755 0)
@@
     )
   )
-  (global_label "VREF_3V3" (shape input) (at 142.24 177.165 0) (fields_autoplaced)
+  (global_label "VREF_3V3" (shape input) (at 142.24 175.895 0) (fields_autoplaced)
     (effects (font (size 1.27 1.27)) (justify left))
-    (property "Intersheetrefs" "${INTERSHEET_REFS}" (at 154.2966 177.165 0)
+    (property "Intersheetrefs" "${INTERSHEET_REFS}" (at 154.2966 175.895 0)
       (effects (font (size 1.27 1.27)) (justify left) hide)
     )
   )
-  (global_label "VREF_1V65" (shape input) (at 88.9 177.165 0) (fields_autoplaced)
+  (global_label "VREF_1V65" (shape input) (at 88.9 175.895 0) (fields_autoplaced)
     (effects (font (size 1.27 1.27)) (justify left))
-    (property "Intersheetrefs" "${INTERSHEET_REFS}" (at 102.1661 177.165 0)
+    (property "Intersheetrefs" "${INTERSHEET_REFS}" (at 102.1661 175.895 0)
       (effects (font (size 1.27 1.27)) (justify left) hide)
     )
@@
       (effects (font (size 1.27 1.27)) hide)
     )
-    (property "Tolerlance" "1%" (at 191.135 90.805 0)
+    (property "Tolerance" "1%" (at 191.135 90.805 0)
       (effects (font (size 1.27 1.27)) hide)
     )
@@
       (effects (font (size 1.27 1.27)) hide)
     )
+    (property "Voltage" "10V" (at 72.39 182.245 0)
+      (effects (font (size 1.27 1.27)) hide)
+    )
     (pin "1")
     (pin "2")
@@
       (effects (font (size 1.27 1.27)))
     )
-    (property "Footprint" "Capacitor_SMD:C_0402_1005Metric_Pad0.74x0.62mm_HandSolder" (at 24.4602 178.435 0)
-      (effects (font (size 1.27 1.27)) hide)
-    )
-    (property "Datasheet" "https://mm.digikey.com/Volume0/opasdata/d220001/medias/docus/609/CL05A105KO5NNNC_Spec_5-2-19.pdf" (at 23.495 182.245 0)
-      (effects (font (size 1.27 1.27)) hide)
-    )
-    (property "Link" "https://www.digikey.com/en/products/detail/samsung-electro-mechanics/CL05A105KO5NNNC/3886725" (at 23.495 182.245 0)
-      (effects (font (size 1.27 1.27)) hide)
-    )
-    (property "Manufacturer" "Samsung Electro-Mechanics" (at 23.495 182.245 0)
-      (effects (font (size 1.27 1.27)) hide)
-    )
-    (property "Manufacturer Number" "CL05A105KO5NNNC" (at 23.495 182.245 0)
-      (effects (font (size 1.27 1.27)) hide)
-    )
-    (property "Tolerance" "10%" (at 23.495 182.245 0)
-      (effects (font (size 1.27 1.27)) hide)
-    )
-    (property "Voltage" "16V" (at 23.495 182.245 0)
-      (effects (font (size 1.27 1.27)) hide)
-    )
-    (property "PCBWay Link" "https://www.pcbway.com/components/detail/CL05A105KO5NNNC/17304/" (at 23.495 182.245 0)
+    (property "Footprint" "Capacitor_SMD:C_0402_1005Metric" (at 24.4602 178.435 0)
+      (effects (font (size 1.27 1.27)) hide)
+    )
+    (property "Datasheet" "https://search.murata.co.jp/Ceramy/image/img/A01X/G101/ENG/GRM155R6YA105KE11-01.pdf" (at 23.495 182.245 0)
+      (effects (font (size 1.27 1.27)) hide)
+    )
+    (property "Link" "https://www.digikey.com/en/products/detail/murata-electronics/GRM155R6YA105KE11J/4905163" (at 23.495 182.245 0)
+      (effects (font (size 1.27 1.27)) hide)
+    )
+    (property "Manufacturer" "Murata Electronics" (at 23.495 182.245 0)
+      (effects (font (size 1.27 1.27)) hide)
+    )
+    (property "Manufacturer Number" "GRM155R6YA105KE11J" (at 23.495 182.245 0)
+      (effects (font (size 1.27 1.27)) hide)
+    )
+    (property "Tolerance" "" (at 23.495 182.245 0)
+      (effects (font (size 1.27 1.27)) hide)
+    )
+    (property "Voltage" "35V" (at 23.495 182.245 0)
+      (effects (font (size 1.27 1.27)) hide)
+    )
+    (property "PCBWay Link" "" (at 23.495 182.245 0)
       (effects (font (size 1.27 1.27)) hide)
     )
@@
       (effects (font (size 1.27 1.27)) hide)
     )
+    (property "Rated Voltage" "35V" (at 23.495 182.245 0)
+      (effects (font (size 1.27 1.27)) hide)
+    )
+    (property "Temperature Coefficient" "X5R" (at 23.495 182.245 0)
+      (effects (font (size 1.27 1.27)) hide)
+    )
