File: hardware/board/sniff_detector/sma_ttl_out.kicad_sch (KiCad schematic)
At the start: 8 parts, among them J7 Conn_Coaxial, U1 74LVCH2T45DC

Commit message: draft firmware
Parts:
- C39: footprint Capacitor_SMD:C_0805_2012Metric -> Capacitor_SMD:C_0603_1608Metric; Alternate CL21B106KOQNNNE -> (none); Link https://www.digikey.com/en/products/detail/murata-electronics/GRM21BZ71E106KE15L/13904911 -> https://www.digikey.com/en/products/detail/murata-electronics/GRM188R61E106KA73J/9887674; Manufacturer Number GRM21BZ71E106KE15L -> GRM188R61E106KA73J; Temperature Coefficient X7R -> X5R; Tolerance (none) -> 10%; Voltage (none) -> 25V
- C53: Tolerance (none) -> 10%; Voltage (none) -> 35V
Changed lines of the file:
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@@
+      (effects (font (size 1.27 1.27)) hide)
+    )
+    (property "Voltage" "35V" (at 141.605 179.07 0)
+      (effects (font (size 1.27 1.27)) hide)
+    )
+    (property "Tolerance" "10%" (at 141.605 179.07 0)
       (effects (font (size 1.27 1.27)) hide)
     )
@@
       (effects (font (size 1.27 1.27)) (justify left))
     )
-    (property "Footprint" "Capacitor_SMD:C_0805_2012Metric" (at 155.9052 182.88 0)
-      (effects (font (size 1.27 1.27)) hide)
-    )
-    (property "Datasheet" "https://search.murata.co.jp/Ceramy/image/img/A01X/G101/ENG/GRM21BZ71E106KE15-01.pdf" (at 154.94 179.07 0)
-      (effects (font (size 1.27 1.27)) hide)
-    )
-    (property "Link" "https://www.digikey.com/en/products/detail/murata-electronics/GRM21BZ71E106KE15L/13904911" (at 154.94 179.07 0)
-      (effects (font (size 1.27 1.27)) hide)
-    )
-    (property "Manufacturer Number" "GRM21BZ71E106KE15L" (at 154.94 179.07 0)
+    (property "Footprint" "Capacitor_SMD:C_0603_1608Metric" (at 155.9052 182.88 0)
+      (effects (font (size 1.27 1.27)) hide)
+    )
+    (property "Datasheet" "https://search.murata.co.jp/Ceramy/image/img/A01X/G101/ENG/GRM188R61E106KA73-01A.pdf" (at 154.94 179.07 0)
+      (effects (font (size 1.27 1.27)) hide)
+    )
+    (property "Link" "https://www.digikey.com/en/products/detail/murata-electronics/GRM188R61E106KA73J/9887674" (at 154.94 179.07 0)
+      (effects (font (size 1.27 1.27)) hide)
+    )
+    (property "Manufacturer Number" "GRM188R61E106KA73J" (at 154.94 179.07 0)
       (effects (font (size 1.27 1.27)) hide)
     )
@@
       (effects (font (size 1.27 1.27)) hide)
     )
-    (property "Temperature Coefficient" "X7R" (at 154.94 179.07 0)
+    (property "Temperature Coefficient" "X5R" (at 154.94 179.07 0)
       (effects (font (size 1.27 1.27)) hide)
     )
@@
       (effects (font (size 1.27 1.27)) hide)
     )
-    (property "Alternate" "CL21B106KOQNNNE" (at 154.94 179.07 0)
-      (effects (font (size 1.27 1.27)) hide)
-    )
+    (property "Alternate" "" (at 154.94 179.07 0)
+      (effects (font (size 1.27 1.27)) hide)
+    )
+    (property "Tolerance" "10%" (at 154.94 179.07 0)
+      (effects (font (size 1.27 1.27)) hide)
+    )
+    (property "Voltage" "25V" (at 154.94 179.07 0)
+      (effects (font (size 1.27 1.27)) hide)
+    )
