File: hardware/board/sniff_detector/sniff_detector.kicad_sch (KiCad schematic)
At the start: 27 parts

Commit message: annotate schematic
Parts:
- C1, C6: value (none) -> 0.1uF; footprint (none) -> Capacitor_SMD:C_0402_1005Metric_Pad0.74x0.62mm_HandSolder
- C2, C3, C9: value (none) -> 10uF; footprint (none) -> Resistor_SMD:R_0603_1608Metric
- C4, C5: value (none) -> 0.1uF; footprint (none) -> Capacitor_SMD:C_1206_3216Metric
- C7: value (none) -> 10uF; footprint (none) -> Capacitor_SMD:C_0805_2012Metric_Pad1.18x1.45mm_HandSolder
- C8: value (none) -> 1uF; footprint (none) -> Capacitor_SMD:C_0402_1005Metric_Pad0.74x0.62mm_HandSolder
- D1: value (none) -> D_Zener; footprint (none) -> Diode_SMD:D_SOD-323
- H1: value (none) -> MountingHole; footprint (none) -> MountingHole:MountingHole_2.7mm
- J1, J2: value (none) -> Conn_01x20_Female; footprint (none) -> Connector_PinHeader_2.54mm:PinHeader_1x20_P2.54mm_Vertical
- J3: value (none) -> Conn_Coaxial; footprint (none) -> Connector_Coaxial:SMA_Samtec_SMA-J-P-X-ST-EM1_EdgeMount
- J4: value (none) -> Conn_01x03_Female; footprint (none) -> Connector_Phoenix_MC:PhoenixContact_MC_1,5_3-G-3.5_1x03_P3.50mm_Horizontal
- JP1, JP2: value (none) -> Jumper_2_Open; footprint (none) -> Jumper:SolderJumper-2_P1.3mm_Open_RoundedPad1.0x1.5mm
- L1: value (none) -> L_Coupled_1423; footprint (none) -> machine_agency_components:L_CommonModeChoke_TDKCorporation_1210
- R1, R2, R3: value (none) -> 22K; footprint (none) -> Resistor_SMD:R_0603_1608Metric
- R4, R5: value (none) -> 15M; footprint (none) -> Resistor_SMD:R_1206_3216Metric
- R6: value (none) -> 470; footprint (none) -> Resistor_SMD:R_0603_1608Metric
- R7: value (none) -> 1K58; footprint (none) -> Resistor_SMD:R_0603_1608Metric
- U1: value (none) -> AD8226; footprint (none) -> Package_SO:MSOP-8_3x3mm_P0.65mm
- U2: value (none) -> REF2033; footprint (none) -> Package_TO_SOT_SMD:SOT-23-5
Other:
- note added: "Common Mode Choke (Optional. Short JP1 & JP2 if L1 is not populated)"
- note added: "Pi Pico switching regulator should be put in PWM mode (GP23 = 1) to reduce switching noise."
- note added: "Pico Bootsel Button Access Hole"
- note removed: "Common Mode Choke (Optional)"
- note removed: "Pi Pico switching regulator should be put in PWM mode to reduce switching noise."
- note removed: "Pico Boot Button Access Hole"
- moved on the sheet: C4, C5, C6, C7, C8, D1, J3, J4, R1, R2, R3, R4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

Commit message: annotate rev1
Parts:
- D1: Manufacturer Number https://www.digikey.com/en/products/detail/nexperia-usa-inc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 -> BZX384-A3V3-QX
Other:
- note added: "FIXME: To reject common mode (60Hz) noise, it would be better to remove the wheatstone configuration."
- note added: "TODO: Does the common mode choke help? Test with the nearby soldering fan turned on/off."
Changed lines of the file:
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@@
     (effects (font (size 1.27 1.27)) (justify left bottom))
+  )
+  (text "TODO: Does the common mode choke help?\nTest with the nearby soldering fan turned on/off."
+    (at 118.11 26.67 0)
+    (effects (font (size 2 2) (thickness 0.254) bold) (justify left bottom))
   )
   (text "22" (at 48.26 78.74 0)
     (effects (font (size 1.27 1.27)) (justify left bottom))
+  )
+  (text "FIXME: To reject common mode (60Hz) noise, it would be\nbetter to remove the wheatstone configuration."
+    (at 74.93 78.74 0)
+    (effects (font (size 1.27 1.27) (thickness 0.254) bold) (justify left bottom))
   )
   (text "VREF has ±20mA output current." (at 245.11 53.34 0)
@@
       (effects (font (size 1.27 1.27)) hide)
     )
-    (property "Datasheet" "~" (id 3) (at 200.66 113.03 0)
-      (effects (font (size 1.27 1.27)) hide)
-    )
-    (property "Manufacturer Number" "https://www.digikey.com/en/products/detail/nexperia-usa-inc/BZX384-A3V3-QX/17295760" (id 4) (at 200.66 113.03 90)
+    (property "Datasheet" "https://assets.nexperia.com/documents/data-sheet/BZX384-Q_SER.pdf" (id 3) (at 200.66 113.03 0)
+      (effects (font (size 1.27 1.27)) hide)
+    )
+    (property "Manufacturer Number" "BZX384-A3V3-QX" (id 4) (at 200.66 113.03 90)
       (effects (font (size 1.27 1.27)) hide)
     )
@@
       (effects (font (size 1.27 1.27)) hide)
     )
+    (property "Field8" "" (id 8) (at 200.66 113.03 90)
+      (effects (font (size 1.27 1.27)) hide)
+    )

Commit message: complete pcb v0.2
Parts:
- removed C1, C6: 0.1uF, Capacitor_SMD:C_0402_1005Metric_Pad0.74x0.62mm_HandSolder, symbol Device:C
- removed C2, C3, C9: 10uF, Resistor_SMD:R_0603_1608Metric, symbol Device:C
- removed C4, C5: 0.1uF, Capacitor_SMD:C_1206_3216Metric, symbol Device:C
- removed C7: 10uF, Capacitor_SMD:C_0805_2012Metric_Pad1.18x1.45mm_HandSolder, symbol Device:C_Polarized
- removed C8: 1uF, Capacitor_SMD:C_0402_1005Metric_Pad0.74x0.62mm_HandSolder, symbol Device:C
- removed D1: D_Zener, Diode_SMD:D_SOD-323, symbol Device:D_Zener
- removed H1: MountingHole, MountingHole:MountingHole_2.7mm, symbol Mechanical:MountingHole
- removed J1, J2: Conn_01x20_Female, Connector_PinHeader_2.54mm:PinHeader_1x20_P2.54mm_Vertical, symbol Connector:Conn_01x20_Female
- removed J3: Conn_Coaxial, Connector_Coaxial:SMA_Samtec_SMA-J-P-X-ST-EM1_EdgeMount, symbol Connector:Conn_Coaxial
- removed J4: Conn_01x03_Female, Connector_Phoenix_MC:PhoenixContact_MC_1,5_3-G-3.5_1x03_P3.50mm_Horizontal, symbol Connector:Conn_01x03_Female
- removed JP1, JP2: Jumper_2_Open, Jumper:SolderJumper-2_P1.3mm_Open_RoundedPad1.0x1.5mm, symbol Jumper:Jumper_2_Open
- removed L1: L_Coupled_1423, machine_agency_components:L_CommonModeChoke_TDKCorporation_1210, symbol Device:L_Coupled_1423
- removed R1, R2, R3: 22K, Resistor_SMD:R_0603_1608Metric, symbol Device:R
- removed R4, R5: 15M, Resistor_SMD:R_1206_3216Metric, symbol Device:R
- removed R6: 470, Resistor_SMD:R_0603_1608Metric, symbol Device:R
- removed R7: 1K58, Resistor_SMD:R_0603_1608Metric, symbol Device:R
- removed U1: AD8226, Package_SO:MSOP-8_3x3mm_P0.65mm, symbol machine_agency_components:AD8226
- removed U2: REF2033, Package_TO_SOT_SMD:SOT-23-5, symbol machine_agency_components:REF20xx
- added H1: MountingHole_Pad, kicad_component_library:Terminal_Keystone_779x_EdgeMount_Horizontal, symbol Mechanical:MountingHole_Pad
Connections:
- net GND: now also H1.1
- no-connect marks 35 -> 0
Other:
- added sheet Harp Core RP2040 + Isolated USB (harp_core_rp2040_w_isolated_usb.kicad_sch)
- added sheet Power Supplies (power_supplies.kicad_sch)
- added sheet Sensing Front End (sensing_front_end.kicad_sch)
- added sheet TTL Output (sma_ttl_out.kicad_sch)
- note added: "External Ground Connection"
- note added: "FIXME: change to "screw-not-supplied" version."
- note removed: "0.1Hz (R = 1M) or 1Hz (R = 100K) Common Mode Highpass Filter"
- note removed: "101Hz Lowpass Filter"
- note removed: "21"
- note removed: "22"
- note removed: "3.3V"
- note removed: "3.3V 1% Clipper"
- note removed: "5V Supply Bypass Cap"
- note removed: "AD8226 configured: * Single Supply (5V) * Bridge Common Mode Voltage: 1.65V * Gain ≈100"
- note removed: "Common Mode Choke (Optional. Short JP1 & JP2 if L1 is not populated)"
- note removed: "FIXME: To reject common mode (60Hz) noise, it would be better to remove the wheatstone configuration."
- note removed: "GNDD"
- note removed: "GP26"
- note removed: "Gain = 106"
- note removed: "High Pass Filter components should be closely matched."
- note removed: "Pi Pico switching regulator should be put in PWM mode (GP23 = 1) to reduce switching noise."
- note removed: "Pico Bootsel Button Access Hole"
- note removed: "Pico Shield Footprint"
- note removed: "REF2033 Input Bypass Cap"
- note removed: "REF2033 Output Bypass Cap"
- note removed: "REF2033 Output/2 Bypass Cap"
- note removed: "Shield →"
- note removed: "TODO: Does the common mode choke help? Test with the nearby soldering fan turned on/off."
- note removed: "Tantalum"
- note removed: "VREF has ±20mA output current."
- note removed: "Wheatstone Bridge"
- note removed: "Wheatstone Bridge fixed resistors should be closely matched."

Commit message: draft firmware
Parts:
- H1: Link https://www.digikey.com/en/products/detail/keystone-electronics/7794/2171012 -> https://www.digikey.com/en/products/detail/keystone-electronics/7792/2171011; Manufacturer Number 7794 -> 7792
Other:
- note removed: "FIXME: change to "screw-not-supplied" version."
Changed lines of the file:
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@@
     (stroke (width 0) (type default))
-  )
-  (text "FIXME: change to \"screw-not-supplied\" version." (at 197.485 132.715 0)
-    (effects (font (size 2 2) (thickness 0.4) bold) (justify left bottom))
   )
   (text "External Ground Connection" (at 247.65 137.16 0)
@@
       (effects (font (size 1.27 1.27)) hide)
     )
-    (property "Datasheet" "n/a" (at 252.73 141.605 0)
+    (property "Datasheet" "https://www.keyelco.com/userAssets/file/M65p69.pdf" (at 252.73 141.605 0)
       (effects (font (size 1.27 1.27)) hide)
     )
-    (property "Link" "https://www.digikey.com/en/products/detail/keystone-electronics/7794/2171012" (at 252.73 141.605 0)
+    (property "Link" "https://www.digikey.com/en/products/detail/keystone-electronics/7792/2171011" (at 252.73 141.605 0)
       (effects (font (size 1.27 1.27)) hide)
     )
@@
       (effects (font (size 1.27 1.27)) hide)
     )
-    (property "Manufacturer Number" "7794" (at 252.73 141.605 0)
+    (property "Manufacturer Number" "7792" (at 252.73 141.605 0)
       (effects (font (size 1.27 1.27)) hide)
     )
